Commit message: Updated Torques and controller tester

File: urdf/Arm_URDF.xacro (robot description, xacro)
@@ -16,5 +16,5 @@
         <mass value = "0.00001" />
         <origin rpy ="0 0 0" xyz ="0 0 0" />
-        <inertia ixx = "0.01" ixy = "0.01" ixz = "0.01" iyy = "0.01" iyz = "0.01" izz = "0.01" />
+        <inertia ixx = "0.0" ixy = "0.0" ixz = "0.0" iyy = "0.0" iyz = "0.0" izz = "0.0" />
     </inertial>
   <joint name="fixed" type="fixed">
@@ -42,5 +42,5 @@
         <child link="arm_base"/>
         <origin xyz="0 0 0.005" rpy="0 0 0"/>
-        <limit lower="-3.14159" upper="3.14159" effort="0.1" velocity="0.005"/>
+        <limit lower="-3.14159" upper="3.14159" effort="5.4917" velocity="0.5"/>
     <axis xyz="0 0 1"/>
 </joint>
@@ -75,5 +75,5 @@
         <child link="arm_lower"/>
         <origin xyz="0 0 0.07" rpy="0 0 0"/>
-        <limit lower="-1.57" upper="1.57" effort="0.1" velocity="0.5"/>
+        <limit lower="-1.57" upper="1.57" effort="5.4917" velocity="0.5"/>
     <axis xyz="1 0 0"/>
 </joint>
@@ -114,5 +114,5 @@
         <child link="arm_upper"/>
         <origin xyz="0 0 0.432" rpy="0 0 0"/>
-        <limit lower="-3.14159" upper="3.14159" effort="0.1" velocity="0.5"/>
+        <limit lower="-3.14159" upper="3.14159" effort="5.4917" velocity="0.5"/>
     <axis xyz="1 0 0"/>
 </joint>
@@ -153,5 +153,5 @@
         <child link="pointer"/>
         <origin xyz="0 0 0.54" rpy="0 0 0"/>
-        <limit lower="-3.14159" upper="3.14159" effort="0.1" velocity="0.5"/>
+        <limit lower="-3.14159" upper="3.14159" effort="5.4917" velocity="0.5"/>
     <axis xyz="1 0 0"/>
 </joint>

Commit message: Updated inertia, collision and spawning properties

File: urdf/Arm_URDF.xacro (robot description, xacro)
@@ -27,5 +27,5 @@
         <mass value = "0.00001" />
         <origin rpy ="0 0 0" xyz ="0 0 0" />
-        <inertia ixx = "0.01" ixy = "0.01" ixz = "0.01" iyy = "0.01" iyz = "0.01" izz = "0.01" />
+        <inertia ixx = "0.00" ixy = "0.00" ixz = "0.00" iyy = "0.00" iyz = "0.00" izz = "0.00" />
     </inertial>
     <visual>
@@ -113,5 +113,5 @@
     <parent link="arm_lower"/>
         <child link="arm_upper"/>
-        <origin xyz="0 0 0.432" rpy="0 0 0"/>
+        <origin xyz="0 0 0.432" rpy="0 0 -3.14"/>
         <limit lower="-3.14159" upper="3.14159" effort="5.4917" velocity="0.5"/>
     <axis xyz="1 0 0"/>
@@ -148,5 +148,5 @@
     </visual>
 </link>
-            <!-- Uper to Pointer Joint -->
+            <!-- Upper to Pointer Joint -->
 <joint name="upper_pointer_joint" type="revolute">
     <parent link="arm_upper"/>

Commit message: Updated angles to match given coordinates

File: urdf/Arm_URDF.xacro (robot description, xacro)
@@ -113,5 +113,5 @@
     <parent link="arm_lower"/>
         <child link="arm_upper"/>
-        <origin xyz="0 0 0.432" rpy="0 0 -3.14"/>
+        <origin xyz="0 0 0.432" rpy="0 0 0"/>
         <limit lower="-3.14159" upper="3.14159" effort="5.4917" velocity="0.5"/>
     <axis xyz="1 0 0"/>
